Commit message: [feat] 调整目录结构，增加机器人urdf

File: robot_model/urdf/include/oak.urdf.xacro (robot description, xacro)
@@ -1,13 +1,9 @@
 <?xml version="1.0"?>
 <robot name="depthai_camera" xmlns:xacro="http://ros.org/wiki/xacro">
-    <xacro:macro name="depthai_camera" params="camera_name camera_model parent base_frame
+    <xacro:macro name="depthai_camera" params="camera_name parent base_frame
                                            cam_pos_x cam_pos_y cam_pos_z
                                            cam_roll cam_pitch cam_yaw
                                            r:=0.8 g:=0.8 b:=0.8 a:=0.8">
         <xacro:property name="M_PI" value="3.1415926535897931"/>
-        <xacro:property name="model" value="${camera_model}"/>
-        <xacro:property name="has_imu" value="false"/>
-        <!-- <xacro:if value="${model == 'BW1098OAK'}">
-        </xacro:if> -->
         <xacro:property name="baseline" value="0.075"/>
         <!-- base_link of the sensor-->
@@ -23,5 +19,5 @@
                 <origin xyz="0 0 0" rpy="0 0 0"/>
                 <geometry>
-                    <mesh filename="package://depthai_bridge/urdf/models/${model}.stl"/>
+                    <mesh filename="package://robot_model/urdf/models/OAK-D-PRO.stl"/>
                 </geometry>
                 <material name="mat">
