Commit message: [feat] 3d->2d投影完成 [misc] 下位机通信协议修改

File: robot/robot_model/urdf/robot.urdf.xacro (robot description, xacro)
@@ -1,10 +1,13 @@
 <?xml version="1.0"?>
 <robot name="robot" xmlns:xacro="http://ros.org/wiki/xacro">
+    <xacro:arg name="prefix"   default="" />
     <xacro:include filename="$(find robot_model)/urdf/include/oak.urdf.xacro"/>
-    <link name="base_link"/>
-    <xacro:depthai_camera camera_name = "oak_front" parent = "base_link" base_frame = "oak_front_frame"
+    <link name="$(arg prefix)base_link"/>
+    <xacro:depthai_camera camera_name = "$(arg prefix)oak_front" parent = "$(arg prefix)base_link"
+                          base_frame = "$(arg prefix)oak_front_frame"
                           cam_pos_x = "0.5" cam_pos_y = "0.0" cam_pos_z = "0.0"
                           cam_roll = "0.0" cam_pitch = "0.0" cam_yaw = "0.0"/>
-    <xacro:depthai_camera camera_name = "oak_back" parent = "base_link" base_frame = "oak_back_frame"
+    <xacro:depthai_camera camera_name = "$(arg prefix)oak_back" parent = "$(arg prefix)base_link"
+                          base_frame = "$(arg prefix)oak_back_frame"
                           cam_pos_x = "-0.5" cam_pos_y = "0.0" cam_pos_z = "0.0"
                           cam_roll = "0.0" cam_pitch = "0.0" cam_yaw = "0.0"/>

Commit message: [update] change 01 day 5

File: robot/robot_model/urdf/robot.urdf.xacro (robot description, xacro)
@@ -12,3 +12,12 @@
                           cam_pos_x = "-0.08" cam_pos_y = "0.0" cam_pos_z = "0.3"
                           cam_roll = "0.0" cam_pitch = "0.0" cam_yaw = "0.0"/>
+    <xacro:macro name="mid360">
+          <link name="$(arg prefix)lidar_body"/>
+          <joint name="$(arg prefix)lidar_joint" type="fixed">
+                  <parent link="$(arg prefix)base_link"/>
+                  <child link="$(arg prefix)lidar_body"/>
+                  <origin xyz="0 0 0.6" rpy="0 0 0"/>
+          </joint>
+    </xacro:macro>
+    <xacro:mid360/>
 </robot>
